Commit message: dfgdfg

File: description/camera.xacro (robot description, xacro)
@@ -1,4 +1,7 @@
 <?xml version="1.0"?>
 <robot xmlns:xacro="http://www.ros.org/wiki/xacro" >
+    <material name="black">
+        <color rgba="0 0 0 0"/>
+    </material>
     <!-- Camera mounted 75mm forward, 100mm above base_link -->
     <joint name="camera_joint" type="fixed">

File: description/lidar.xacro (robot description, xacro)
@@ -2,4 +2,7 @@
 <robot xmlns:xacro="http://www.ros.org/wiki/xacro" >
     <xacro:include filename="inertial_macros.xacro"/>
+    <material name="black">
+        <color rgba="0 0 0 0"/>
+    </material>
     <!-- LiDAR mounted at geometric center, 200mm above base_link -->
     <joint name="laser_joint" type="fixed">

Commit message: fgh

File: description/camera.xacro (robot description, xacro)
@@ -1,7 +1,4 @@
 <?xml version="1.0"?>
 <robot xmlns:xacro="http://www.ros.org/wiki/xacro" >
-    <material name="black">
-        <color rgba="0 0 0 0"/>
-    </material>
     <!-- Camera mounted 75mm forward, 100mm above base_link -->
     <joint name="camera_joint" type="fixed">

File: description/lidar.xacro (robot description, xacro)
@@ -2,7 +2,4 @@
 <robot xmlns:xacro="http://www.ros.org/wiki/xacro" >
     <xacro:include filename="inertial_macros.xacro"/>
-    <material name="black">
-        <color rgba="0 0 0 0"/>
-    </material>
     <!-- LiDAR mounted at geometric center, 200mm above base_link -->
     <joint name="laser_joint" type="fixed">
